File: quasi_nano_led.brd (EAGLE design)
At the start: 40.3 x 58.4 mm, 4 parts, among them X1 JST-XH-02-PIN-LONG-PAD

Commit message: update
Parts:
- moved X1 1.27 mm to (19.1, 29.2)
Routing:
- net N$4: track 40.9 -> 40.3 mm
Other:
- board size 40.3 x 58.4 mm -> 32.7 x 52.1 mm
Changed lines of the file:
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@@
 <board>
 <plain>
-<wire x1="2.54" y1="21.59" x2="42.85" y2="21.59" width="0" layer="20"/>
-<wire x1="42.85" y1="21.59" x2="42.85" y2="80" width="0" layer="20"/>
-<wire x1="42.85" y1="80" x2="2.54" y2="80" width="0" layer="20"/>
-<wire x1="2.54" y1="80" x2="2.54" y2="21.59" width="0" layer="20"/>
+<wire x1="7.62" y1="24.13" x2="40.31" y2="24.13" width="0" layer="20"/>
+<wire x1="40.31" y1="24.13" x2="40.31" y2="76.19" width="0" layer="20"/>
+<wire x1="40.31" y1="76.19" x2="7.62" y2="76.19" width="0" layer="20"/>
+<wire x1="7.62" y1="76.19" x2="7.62" y2="24.13" width="0" layer="20"/>
 </plain>
 <attributes>
@@
 <attribute name="NAME" x="30.3175" y="50.9425" size="0.8128" layer="25" font="vector"/>
 </element>
-<element name="X1" library="Rembrandt Electronics - JST XH Connectors v1-0" package="JST-XH-02-PACKAGE-LONG-PAD" value="JST-XH-02-PIN-LONG-PAD" x="19.05" y="27.94" smashed="yes">
-<attribute name="NAME" x="14.795" y="25.9" size="1.016" layer="25" ratio="10" rot="R90"/>
-<attribute name="VALUE" x="15.7475" y="31.8325" size="1.016" layer="27" ratio="10"/>
+<element name="X1" library="Rembrandt Electronics - JST XH Connectors v1-0" package="JST-XH-02-PACKAGE-LONG-PAD" value="JST-XH-02-PIN-LONG-PAD" x="19.05" y="29.21" smashed="yes">
+<attribute name="NAME" x="14.795" y="27.17" size="1.016" layer="25" ratio="10" rot="R90"/>
+<attribute name="VALUE" x="15.7475" y="33.1025" size="1.016" layer="27" ratio="10"/>
 </element>
 </elements>
@@
 <contactref element="X1" pad="2"/>
 <wire x1="36.3175" y1="58.4675" x2="36.3175" y2="48.3075" width="1.016" layer="16"/>
-<wire x1="36.3175" y1="37.5875" x2="26.67" y2="27.94" width="1.016" layer="16"/>
-<wire x1="26.67" y1="27.94" x2="20.32" y2="27.94" width="1.016" layer="16"/>
+<wire x1="36.3175" y1="37.5875" x2="27.94" y2="29.21" width="1.016" layer="16"/>
+<wire x1="27.94" y1="29.21" x2="20.32" y2="29.21" width="1.016" layer="16"/>
 <wire x1="36.3175" y1="48.3075" x2="36.3175" y2="37.5875" width="1.016" layer="16"/>
 </signal>
@@
 <polygon width="0.1524" layer="16" isolate="0.8128">
 <vertex x="0" y="82.55"/>
-<vertex x="45.72" y="82.55"/>
-<vertex x="45.72" y="20.32"/>
-<vertex x="0" y="20.32"/>
+<vertex x="46.99" y="82.55"/>
+<vertex x="46.99" y="17.78"/>
+<vertex x="0" y="17.78"/>
 </polygon>
 <contactref element="X1" pad="1"/>

Commit message: updated board
Parts:
- removed U$4, U$5: JST-PH_3-PIN_HEADER, con-jst-ph:JST_B3B-PH_HEADER
- added X2, X3: JST-XH-03-PIN-LONG-PAD, Rembrandt Electronics - JST XH Connectors v1-0:JST-XH-03-PACKAGE-LONG-PAD
Connections:
- net GND: now also X2.3, X3.3; no longer U$4.P3, U$5.P3
- net N$4: now also X2.1, X3.1; no longer U$4.P1, U$5.P1
- net N$6: now also X2.2; no longer U$4.P2
- net N$7: now also X3.2; no longer U$5.P2
Routing:
- net N$4: track 40.3 -> 43.8 mm
- net N$6: track 10.2 -> 7.02 mm
- net N$7: track 10.1 -> 12.7 mm
Other:
- board size 32.7 x 52.1 mm -> 32.2 x 53.3 mm
Changed lines of the file:
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@@
 <setting verticaltext="up"/>
 </settings>
-<grid distance="50" unitdist="mil" unit="mil" style="lines" multiple="1" display="no" altdistance="5" altunitdist="mil" altunit="mil"/>
+<grid distance="10" unitdist="mil" unit="mil" style="lines" multiple="10" display="no" altdistance="5" altunitdist="mil" altunit="mil"/>
 <layers>
 <layer number="1" name="Top" color="4" fill="1" visible="yes" active="yes"/>
@@
 <board>
 <plain>
-<wire x1="7.62" y1="24.13" x2="40.31" y2="24.13" width="0" layer="20"/>
-<wire x1="40.31" y1="24.13" x2="40.31" y2="76.19" width="0" layer="20"/>
-<wire x1="40.31" y1="76.19" x2="7.62" y2="76.19" width="0" layer="20"/>
-<wire x1="7.62" y1="76.19" x2="7.62" y2="24.13" width="0" layer="20"/>
+<wire x1="7.62" y1="24.13" x2="39.802" y2="24.13" width="0" layer="20"/>
+<wire x1="39.802" y1="24.13" x2="39.802" y2="77.46" width="0" layer="20"/>
+<wire x1="39.802" y1="77.46" x2="7.62" y2="77.46" width="0" layer="20"/>
+<wire x1="7.62" y1="77.46" x2="7.62" y2="24.13" width="0" layer="20"/>
 </plain>
 <attributes>
@@
 <elements>
 <element name="U$1" library="Arduino-clone" package="NANO" value="NANO" x="21.59" y="46.99" smashed="yes"/>
-<element name="U$4" library="con-jst-ph" package="JST_B3B-PH_HEADER" value="JST-PH_3-PIN_HEADER" x="34.29" y="58.42" smashed="yes">
-<attribute name="NAME" x="30.3175" y="61.1025" size="0.8128" layer="25" font="vector"/>
-</element>
-<element name="U$5" library="con-jst-ph" package="JST_B3B-PH_HEADER" value="JST-PH_3-PIN_HEADER" x="34.29" y="48.26" smashed="yes">
-<attribute name="NAME" x="30.3175" y="50.9425" size="0.8128" layer="25" font="vector"/>
-</element>
 <element name="X1" library="Rembrandt Electronics - JST XH Connectors v1-0" package="JST-XH-02-PACKAGE-LONG-PAD" value="JST-XH-02-PIN-LONG-PAD" x="19.05" y="29.21" smashed="yes">
 <attribute name="NAME" x="14.795" y="27.17" size="1.016" layer="25" ratio="10" rot="R90"/>
 <attribute name="VALUE" x="15.7475" y="33.1025" size="1.016" layer="27" ratio="10"/>
 </element>
+<element name="X2" library="Rembrandt Electronics - JST XH Connectors v1-0" package="JST-XH-03-PACKAGE-LONG-PAD" value="JST-XH-03-PIN-LONG-PAD" x="33.274" y="56.896" smashed="yes" rot="R90">
+<attribute name="NAME" x="35.314" y="51.341" size="1.016" layer="25" ratio="10" rot="R180"/>
+<attribute name="VALUE" x="29.3815" y="52.2935" size="1.016" layer="27" ratio="10" rot="R90"/>
+</element>
+<element name="X3" library="Rembrandt Electronics - JST XH Connectors v1-0" package="JST-XH-03-PACKAGE-LONG-PAD" value="JST-XH-03-PIN-LONG-PAD" x="33.02" y="44.45" smashed="yes" rot="R270">
+<attribute name="NAME" x="30.98" y="50.005" size="1.016" layer="25" ratio="10"/>
+<attribute name="VALUE" x="36.9125" y="49.0525" size="1.016" layer="27" ratio="10" rot="R270"/>
+</element>
 </elements>
 <signals>
 <signal name="N$4">
-<contactref element="U$4" pad="P1"/>
-<contactref element="U$5" pad="P1"/>
 <contactref element="X1" pad="2"/>
-<wire x1="36.3175" y1="58.4675" x2="36.3175" y2="48.3075" width="1.016" layer="16"/>
-<wire x1="36.3175" y1="37.5875" x2="27.94" y2="29.21" width="1.016" layer="16"/>
-<wire x1="27.94" y1="29.21" x2="20.32" y2="29.21" width="1.016" layer="16"/>
-<wire x1="36.3175" y1="48.3075" x2="36.3175" y2="37.5875" width="1.016" layer="16"/>
+<wire x1="20.32" y1="29.21" x2="27.94" y2="29.21" width="1.016" layer="16"/>
+<contactref element="X3" pad="1"/>
+<contactref element="X2" pad="1"/>
+<wire x1="36.83" y1="38.1" x2="36.83" y2="46.99" width="1.016" layer="16"/>
+<wire x1="36.83" y1="46.99" x2="36.83" y2="54.356" width="1.016" layer="16"/>
+<wire x1="36.83" y1="54.356" x2="33.274" y2="54.356" width="1.016" layer="16"/>
+<wire x1="27.94" y1="29.21" x2="36.83" y2="38.1" width="1.016" layer="16"/>
+<wire x1="33.02" y1="46.99" x2="36.83" y2="46.99" width="1.016" layer="16"/>
 </signal>
 <signal name="N$6">
-<contactref element="U$4" pad="P2"/>
 <contactref element="U$1" pad="D5"/>
-<wire x1="26.67" y1="55.88" x2="34.3175" y2="55.88" width="0.6096" layer="16"/>
-<wire x1="34.3175" y1="55.88" x2="34.3175" y2="58.4675" width="0.6096" layer="16"/>
+<contactref element="X2" pad="2"/>
+<wire x1="26.67" y1="55.88" x2="30.48" y2="55.88" width="0.6096" layer="16"/>
+<wire x1="30.48" y1="55.88" x2="31.496" y2="56.896" width="0.6096" layer="16"/>
+<wire x1="31.496" y1="56.896" x2="33.274" y2="56.896" width="0.6096" layer="16"/>
 </signal>
 <signal name="N$7">
 <contactref element="U$1" pad="D3"/>
-<contactref element="U$5" pad="P2"/>
-<wire x1="34.3175" y1="48.3075" x2="34.3175" y2="50.8" width="0.6096" layer="16"/>
-<wire x1="34.3175" y1="50.8" x2="26.67" y2="50.8" width="0.6096" layer="16"/>
+<contactref element="X3" pad="2"/>
+<wire x1="30.226" y1="50.8" x2="26.67" y2="50.8" width="0.6096" layer="16"/>
+<wire x1="33.02" y1="44.45" x2="30.226" y2="44.45" width="0.6096" layer="16"/>
+<wire x1="30.226" y1="44.45" x2="30.226" y2="50.8" width="0.6096" layer="16"/>
 </signal>
 <signal name="GND">
@@
 <contactref element="X1" pad="1"/>
 <contactref element="U$1" pad="GND"/>
-<contactref element="U$5" pad="P3"/>
-<contactref element="U$4" pad="P3"/>
 <contactref element="U$1" pad="GND1"/>
+<contactref element="X3" pad="3"/>
+<contactref element="X2" pad="3"/>
 </signal>
 </signals>
