File: quasi_nano_led.sch (EAGLE design)
At the start: 4 parts, among them X1 JST-XH-02-PIN-LONG-PAD

Commit message: updated board
Parts:
- removed U$4, U$5: JST-PH_3-PIN_HEADER, con-jst-ph:JST-PH_3-PIN_HEADER
- added X2, X3: JST-XH-03-PIN-LONG-PAD, Rembrandt Electronics - JST XH Connectors v1-0:JST-XH-03-PIN-LONG-PAD
Connections:
- net GND: now also X2-3.S, X3-3.S; no longer U$4.3, U$5.3
- net N$4: now also X2-1.S, X3-1.S; no longer U$4.1, U$5.1
- net N$6: now also X2-2.S; no longer U$4.2
- net N$7: now also X3-2.S; no longer U$5.2
Changed lines of the file:
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@@
 <parts>
 <part name="U$1" library="Arduino-clone" deviceset="NANO" device=""/>
-<part name="U$4" library="con-jst-ph" deviceset="JST-PH_3-PIN_HEADER" device=""/>
-<part name="U$5" library="con-jst-ph" deviceset="JST-PH_3-PIN_HEADER" device=""/>
 <part name="X1" library="Rembrandt Electronics - JST XH Connectors v1-0" deviceset="JST-XH-02-PIN" device="-LONG-PAD"/>
+<part name="X2" library="Rembrandt Electronics - JST XH Connectors v1-0" deviceset="JST-XH-03-PIN" device="-LONG-PAD"/>
+<part name="X3" library="Rembrandt Electronics - JST XH Connectors v1-0" deviceset="JST-XH-03-PIN" device="-LONG-PAD"/>
 </parts>
 <sheets>
@@
 <instances>
 <instance part="U$1" gate="G$1" x="53.34" y="66.04" smashed="yes"/>
-<instance part="U$4" gate="G$1" x="83.82" y="71.12" smashed="yes">
-<attribute name="NAME" x="81.28" y="76.962" size="1.27" layer="95"/>
-<attribute name="VALUE" x="81.28" y="64.262" size="1.27" layer="96"/>
-</instance>
-<instance part="U$5" gate="G$1" x="88.9" y="55.88" smashed="yes">
-<attribute name="NAME" x="86.36" y="61.722" size="1.27" layer="95"/>
-<attribute name="VALUE" x="86.36" y="49.022" size="1.27" layer="96"/>
-</instance>
 <instance part="X1" gate="-2" x="27.94" y="96.52" smashed="yes">
 <attribute name="NAME" x="30.48" y="95.758" size="1.524" layer="95"/>
@@
 <attribute name="NAME" x="30.48" y="98.298" size="1.524" layer="95"/>
 <attribute name="VALUE" x="27.178" y="100.457" size="1.778" layer="96"/>
+</instance>
+<instance part="X2" gate="-1" x="83.82" y="83.82" smashed="yes">
+<attribute name="NAME" x="86.36" y="83.058" size="1.524" layer="95"/>
+<attribute name="VALUE" x="83.058" y="85.217" size="1.778" layer="96"/>
+</instance>
+<instance part="X2" gate="-2" x="83.82" y="81.28" smashed="yes">
+<attribute name="NAME" x="86.36" y="80.518" size="1.524" layer="95"/>
+</instance>
+<instance part="X2" gate="-3" x="83.82" y="78.74" smashed="yes">
+<attribute name="NAME" x="86.36" y="77.978" size="1.524" layer="95"/>
+</instance>
+<instance part="X3" gate="-1" x="99.06" y="58.42" smashed="yes">
+<attribute name="NAME" x="101.6" y="57.658" size="1.524" layer="95"/>
+<attribute name="VALUE" x="98.298" y="59.817" size="1.778" layer="96"/>
+</instance>
+<instance part="X3" gate="-2" x="99.06" y="55.88" smashed="yes">
+<attribute name="NAME" x="101.6" y="55.118" size="1.524" layer="95"/>
+</instance>
+<instance part="X3" gate="-3" x="99.06" y="53.34" smashed="yes">
+<attribute name="NAME" x="101.6" y="52.578" size="1.524" layer="95"/>
 </instance>
 </instances>
@@
 <segment>
 <wire x1="25.4" y1="88.9" x2="71.12" y2="88.9" width="0.1524" layer="91"/>
-<pinref part="U$4" gate="G$1" pin="1"/>
 <wire x1="78.74" y1="73.66" x2="71.12" y2="73.66" width="0.1524" layer="91"/>
 <wire x1="71.12" y1="73.66" x2="71.12" y2="88.9" width="0.1524" layer="91"/>
-<pinref part="U$5" gate="G$1" pin="1"/>
-<wire x1="83.82" y1="58.42" x2="71.12" y2="58.42" width="0.1524" layer="91"/>
+<wire x1="96.52" y1="58.42" x2="71.12" y2="58.42" width="0.1524" layer="91"/>
 <wire x1="71.12" y1="58.42" x2="71.12" y2="73.66" width="0.1524" layer="91"/>
 <junction x="71.12" y="73.66"/>
 <pinref part="X1" gate="-2" pin="S"/>
 <wire x1="25.4" y1="96.52" x2="25.4" y2="88.9" width="0.1524" layer="91"/>
+<pinref part="X3" gate="-1" pin="S"/>
+<pinref part="X2" gate="-1" pin="S"/>
+<wire x1="81.28" y1="83.82" x2="78.74" y2="83.82" width="0.1524" layer="91"/>
+<wire x1="78.74" y1="83.82" x2="78.74" y2="73.66" width="0.1524" layer="91"/>
 </segment>
 </net>
 <net name="N$6" class="0">
 <segment>
-<pinref part="U$4" gate="G$1" pin="2"/>
-<wire x1="78.74" y1="71.12" x2="76.2" y2="71.12" width="0.1524" layer="91"/>
 <wire x1="76.2" y1="71.12" x2="76.2" y2="63.5" width="0.1524" layer="91"/>
 <pinref part="U$1" gate="G$1" pin="D5"/>
 <wire x1="76.2" y1="63.5" x2="63.5" y2="63.5" width="0.1524" layer="91"/>
+<wire x1="76.2" y1="71.12" x2="81.28" y2="71.12" width="0.1524" layer="91"/>
+<wire x1="81.28" y1="71.12" x2="81.28" y2="76.2" width="0.1524" layer="91"/>
+<wire x1="81.28" y1="76.2" x2="73.66" y2="76.2" width="0.1524" layer="91"/>
+<wire x1="73.66" y1="76.2" x2="73.66" y2="81.28" width="0.1524" layer="91"/>
+<pinref part="X2" gate="-2" pin="S"/>
+<wire x1="73.66" y1="81.28" x2="81.28" y2="81.28" width="0.1524" layer="91"/>
 </segment>
 </net>
@@
 <wire x1="63.5" y1="58.42" x2="68.58" y2="58.42" width="0.1524" layer="91"/>
 <wire x1="68.58" y1="58.42" x2="68.58" y2="55.88" width="0.1524" layer="91"/>
-<pinref part="U$5" gate="G$1" pin="2"/>
-<wire x1="68.58" y1="55.88" x2="83.82" y2="55.88" width="0.1524" layer="91"/>
+<wire x1="68.58" y1="55.88" x2="96.52" y2="55.88" width="0.1524" layer="91"/>
+<pinref part="X3" gate="-2" pin="S"/>
 </segment>
 </net>
@@
 </segment>
 <segment>
-<pinref part="U$5" gate="G$1" pin="3"/>
-<wire x1="83.82" y1="53.34" x2="78.74" y2="53.34" width="0.1524" layer="91"/>
+<wire x1="96.52" y1="53.34" x2="78.74" y2="53.34" width="0.1524" layer="91"/>
 <label x="78.74" y="53.34" size="1.778" layer="95"/>
+<pinref part="X3" gate="-3" pin="S"/>
 </segment>
 <segment>
-<pinref part="U$4" gate="G$1" pin="3"/>
-<wire x1="78.74" y1="68.58" x2="73.66" y2="68.58" width="0.1524" layer="91"/>
 <label x="73.66" y="68.58" size="1.778" layer="95"/>
+<pinref part="X2" gate="-3" pin="S"/>
+<wire x1="81.28" y1="78.74" x2="76.2" y2="78.74" width="0.1524" layer="91"/>
+<wire x1="81.28" y1="78.74" x2="83.82" y2="78.74" width="0.1524" layer="91"/>
+<wire x1="83.82" y1="78.74" x2="83.82" y2="68.58" width="0.1524" layer="91"/>
+<wire x1="83.82" y1="68.58" x2="73.66" y2="68.58" width="0.1524" layer="91"/>
 </segment>
 <segment>
